Commit message: Make wheel rotation visible in RViz

File: joystick/ros2_ws/src/rhylon_joystick/urdf/rhylon_car.urdf (robot description, URDF)
Before this commit: robot rhylon_car, 6 links, 5 joints
Links:
- link front_left_wheel: geometry visual box size=0.010 0.012 0.006; visual cylinder length=0.016 radius=0.024
- link front_right_wheel: geometry visual box size=0.010 0.012 0.006; visual cylinder length=0.016 radius=0.024
- link rear_left_wheel: geometry visual box size=0.010 0.012 0.006; visual cylinder length=0.016 radius=0.024
- link rear_right_wheel: geometry visual box size=0.010 0.012 0.006; visual cylinder length=0.016 radius=0.024

Commit message: Use spoke-style wheel visuals for RViz

File: joystick/ros2_ws/src/rhylon_joystick/urdf/rhylon_car.urdf (robot description, URDF)
Before this commit: robot rhylon_car, 6 links, 5 joints
Links:
- link front_left_wheel: geometry visual box size=0.006 0.010 0.018; visual box size=0.006 0.010 0.018
- link front_right_wheel: geometry visual box size=0.006 0.010 0.018; visual box size=0.006 0.010 0.018
- link rear_left_wheel: geometry visual box size=0.006 0.010 0.018; visual box size=0.006 0.010 0.018
- link rear_right_wheel: geometry visual box size=0.006 0.010 0.018; visual box size=0.006 0.010 0.018
